File: Ki Cad PCB.kicad_sch (KiCad schematic)
At the start: 137 parts

Commit message: Ki Cad Schematic for PCB
Parts:
- D_#1: renamed from D_#; footprint (none) -> keyboard_parts:D_SOD123_axial
- D_'1: renamed from D_'; footprint (none) -> keyboard_parts:D_SOD123_axial
- D_,1: renamed from D_,; footprint (none) -> keyboard_parts:D_SOD123_axial
- D_-1: renamed from D_-; footprint (none) -> keyboard_parts:D_SOD123_axial
- D_.1: renamed from D_.; footprint (none) -> keyboard_parts:D_SOD123_axial
- D_/1: renamed from D_/; footprint (none) -> keyboard_parts:D_SOD123_axial
- D_0, D_1, D_2, D_3, D_4, D_5, D_6, D_7, D_8, D_9, D_MAC1, D_MAC2, D_MAC3, D_MAC4, D_SHIFT2: footprint (none) -> keyboard_parts:D_SOD123_axial
- D_;1: renamed from D_;; footprint (none) -> keyboard_parts:D_SOD123_axial
- D_=1: renamed from D_=; footprint (none) -> keyboard_parts:D_SOD123_axial
- D_A1: renamed from D_A; footprint (none) -> keyboard_parts:D_SOD123_axial
- D_ALT1, D_ALT2: renamed from D_ALT; footprint (none) -> keyboard_parts:D_SOD123_axial
- D_B1: renamed from D_B; footprint (none) -> keyboard_parts:D_SOD123_axial
- D_BACK1: renamed from D_BACK; footprint (none) -> keyboard_parts:D_SOD123_axial
- D_C1: renamed from D_C; footprint (none) -> keyboard_parts:D_SOD123_axial
- D_CAPS1: renamed from D_CAPS; footprint (none) -> keyboard_parts:D_SOD123_axial
- D_CTRL1: renamed from D_CTRL; footprint (none) -> keyboard_parts:D_SOD123_axial
- D_D1: renamed from D_D; footprint (none) -> keyboard_parts:D_SOD123_axial
- D_DOWN1: renamed from D_DOWN; footprint (none) -> keyboard_parts:D_SOD123_axial
- D_E1: renamed from D_E; footprint (none) -> keyboard_parts:D_SOD123_axial
- D_ENTER1: renamed from D_ENTER; footprint (none) -> keyboard_parts:D_SOD123_axial
- D_ESC1: renamed from D_ESC; footprint (none) -> keyboard_parts:D_SOD123_axial
- D_F1: renamed from D_F; footprint (none) -> keyboard_parts:D_SOD123_axial
- D_FN1, D_WINDOWS1: renamed from D_WINDOWS; footprint (none) -> keyboard_parts:D_SOD123_axial
- D_G1: renamed from D_G; footprint (none) -> keyboard_parts:D_SOD123_axial
- D_H1: renamed from D_H; footprint (none) -> keyboard_parts:D_SOD123_axial
- D_I1: renamed from D_I; footprint (none) -> keyboard_parts:D_SOD123_axial
- D_J1: renamed from D_J; footprint (none) -> keyboard_parts:D_SOD123_axial
- D_K1: renamed from D_K; footprint (none) -> keyboard_parts:D_SOD123_axial
- D_L1: renamed from D_L; footprint (none) -> keyboard_parts:D_SOD123_axial
- D_LEFT1: renamed from D_LEFT; footprint (none) -> keyboard_parts:D_SOD123_axial
- D_M1: renamed from D_M; footprint (none) -> keyboard_parts:D_SOD123_axial
- D_MENU1: renamed from D_MENU; footprint (none) -> keyboard_parts:D_SOD123_axial
- D_N1: renamed from D_N; footprint (none) -> keyboard_parts:D_SOD123_axial
- D_O1: renamed from D_O; footprint (none) -> keyboard_parts:D_SOD123_axial
- D_P1: renamed from D_P; footprint (none) -> keyboard_parts:D_SOD123_axial
- D_Q1: renamed from D_Q; footprint (none) -> keyboard_parts:D_SOD123_axial
- D_R1: renamed from D_R; footprint (none) -> keyboard_parts:D_SOD123_axial
- D_RIGHTY1: renamed from D_RIGHTY; footprint (none) -> keyboard_parts:D_SOD123_axial
- D_S1: renamed from D_S; footprint (none) -> keyboard_parts:D_SOD123_axial
- D_SHIFT1: renamed from D_SHIFT; footprint (none) -> keyboard_parts:D_SOD123_axial
- D_SPACEBAR1: renamed from D_SPACEBAR; footprint (none) -> keyboard_parts:D_SOD123_axial
- D_T1: renamed from D_T; footprint (none) -> keyboard_parts:D_SOD123_axial
- D_TAB1: renamed from D_TAB; footprint (none) -> keyboard_parts:D_SOD123_axial
- D_U1: renamed from D_U; footprint (none) -> keyboard_parts:D_SOD123_axial
- D_UP1: renamed from D_UP; footprint (none) -> keyboard_parts:D_SOD123_axial
- D_V1: renamed from D_V; footprint (none) -> keyboard_parts:D_SOD123_axial
- D_W1: renamed from D_W; footprint (none) -> keyboard_parts:D_SOD123_axial
- D_X1: renamed from D_X; footprint (none) -> keyboard_parts:D_SOD123_axial
- D_Y1: renamed from D_Y; footprint (none) -> keyboard_parts:D_SOD123_axial
- D_Z1: renamed from D_Z; footprint (none) -> keyboard_parts:D_SOD123_axial
- D_[1: renamed from D_[; footprint (none) -> keyboard_parts:D_SOD123_axial
- D_]1: renamed from D_]; footprint (none) -> keyboard_parts:D_SOD123_axial
- K_#1: renamed from K_#; footprint (none) -> Button_Switch_Keyboard:SW_Cherry_MX_1.50u_Plate
- K_'1: renamed from K_'; footprint (none) -> Button_Switch_Keyboard:SW_Cherry_MX_1.00u_Plate
- K_,1: renamed from K_,; footprint (none) -> Button_Switch_Keyboard:SW_Cherry_MX_1.00u_Plate
- K_-1: renamed from K_-; footprint (none) -> Button_Switch_Keyboard:SW_Cherry_MX_1.00u_Plate
- K_.1: renamed from K_.; footprint (none) -> Button_Switch_Keyboard:SW_Cherry_MX_1.00u_Plate
- K_/1: renamed from K_/; footprint (none) -> Button_Switch_Keyboard:SW_Cherry_MX_1.00u_Plate
- K_0, K_1, K_2, K_3, K_4, K_5, K_6, K_7, K_8, K_9, K_MAC1, K_MAC2, K_MAC3, K_MAC4: footprint (none) -> Button_Switch_Keyboard:SW_Cherry_MX_1.00u_Plate
- K_;1: renamed from K_;; footprint (none) -> Button_Switch_Keyboard:SW_Cherry_MX_1.00u_Plate
- K_=1: renamed from K_=; footprint (none) -> Button_Switch_Keyboard:SW_Cherry_MX_1.00u_Plate
- K_A1: renamed from K_A; footprint (none) -> Button_Switch_Keyboard:SW_Cherry_MX_1.00u_Plate
- K_ALT1, K_ALT2: renamed from K_ALT; footprint (none) -> Button_Switch_Keyboard:SW_Cherry_MX_1.25u_Plate
- K_B1: renamed from K_B; footprint (none) -> Button_Switch_Keyboard:SW_Cherry_MX_1.00u_Plate
- K_BACK1: renamed from K_BACK; footprint (none) -> Button_Switch_Keyboard:SW_Cherry_MX_2.00u_Plate
- K_C1: renamed from K_C; footprint (none) -> Button_Switch_Keyboard:SW_Cherry_MX_1.00u_Plate
- K_CAPS1: renamed from K_CAPS; footprint (none) -> Button_Switch_Keyboard:SW_Cherry_MX_1.75u_Plate
- K_CTRL1, K_CTRL2: renamed from K_CTRL; footprint (none) -> Button_Switch_Keyboard:SW_Cherry_MX_1.25u_Plate
- K_D1: renamed from K_D; footprint (none) -> Button_Switch_Keyboard:SW_Cherry_MX_1.00u_Plate
- K_DOWN1: renamed from K_DOWN; footprint (none) -> Button_Switch_Keyboard:SW_Cherry_MX_1.00u_Plate
- K_E1: renamed from K_E; footprint (none) -> Button_Switch_Keyboard:SW_Cherry_MX_1.00u_Plate
- K_ENTER1: renamed from K_ENTER; footprint (none) -> Button_Switch_Keyboard:SW_Cherry_MX_2.25u_Plate
- K_ESC1: renamed from K_ESC; footprint (none) -> Button_Switch_Keyboard:SW_Cherry_MX_1.00u_Plate
- K_F1: renamed from K_F; footprint (none) -> Button_Switch_Keyboard:SW_Cherry_MX_1.00u_Plate
- K_FN1, K_WINDOWS1: renamed from K_WINDOWS; footprint (none) -> Button_Switch_Keyboard:SW_Cherry_MX_1.25u_Plate
- K_G1: renamed from K_G; footprint (none) -> Button_Switch_Keyboard:SW_Cherry_MX_1.00u_Plate
- K_H1: renamed from K_H; footprint (none) -> Button_Switch_Keyboard:SW_Cherry_MX_1.00u_Plate
- K_I1: renamed from K_I; footprint (none) -> Button_Switch_Keyboard:SW_Cherry_MX_1.00u_Plate
- K_J1: renamed from K_J; footprint (none) -> Button_Switch_Keyboard:SW_Cherry_MX_1.00u_Plate
- K_K1: renamed from K_K; footprint (none) -> Button_Switch_Keyboard:SW_Cherry_MX_1.00u_Plate
- K_L1: renamed from K_L; footprint (none) -> Button_Switch_Keyboard:SW_Cherry_MX_1.00u_Plate
- K_LEFT1: renamed from K_LEFT; footprint (none) -> Button_Switch_Keyboard:SW_Cherry_MX_1.00u_Plate
- K_M1: renamed from K_M; footprint (none) -> Button_Switch_Keyboard:SW_Cherry_MX_1.00u_Plate
- K_N1: renamed from K_N; footprint (none) -> Button_Switch_Keyboard:SW_Cherry_MX_1.00u_Plate
- K_O1: renamed from K_O; footprint (none) -> Button_Switch_Keyboard:SW_Cherry_MX_1.00u_Plate
- K_P1: renamed from K_P; footprint (none) -> Button_Switch_Keyboard:SW_Cherry_MX_1.00u_Plate
- K_Q1: renamed from K_Q; footprint (none) -> Button_Switch_Keyboard:SW_Cherry_MX_1.00u_Plate
- K_R1: renamed from K_R; footprint (none) -> Button_Switch_Keyboard:SW_Cherry_MX_1.00u_Plate
- K_RIGHT1: renamed from K_RIGHT; footprint (none) -> Button_Switch_Keyboard:SW_Cherry_MX_1.00u_Plate
- K_S1: renamed from K_S; footprint (none) -> Button_Switch_Keyboard:SW_Cherry_MX_1.00u_Plate
- K_SHIFT1: renamed from K_SHIFT; footprint (none) -> Button_Switch_Keyboard:SW_Cherry_MX_2.25u_Plate
- K_SHIFT2: footprint (none) -> Button_Switch_Keyboard:SW_Cherry_MX_2.75u_Plate
- K_SPACEBARD1: renamed from K_SPACEBARD; footprint (none) -> Button_Switch_Keyboard:SW_Cherry_MX_6.25u_Plate
- K_T1: renamed from K_T; footprint (none) -> Button_Switch_Keyboard:SW_Cherry_MX_1.00u_PCB
- K_TAB1: renamed from K_TAB; footprint (none) -> Button_Switch_Keyboard:SW_Cherry_MX_1.50u_Plate
- K_U1: renamed from K_U; footprint (none) -> Button_Switch_Keyboard:SW_Cherry_MX_1.00u_Plate
- K_UP1: renamed from K_UP; footprint (none) -> Button_Switch_Keyboard:SW_Cherry_MX_1.00u_Plate
- K_V1: renamed from K_V; footprint (none) -> Button_Switch_Keyboard:SW_Cherry_MX_1.00u_Plate
- K_W1: renamed from K_W; footprint (none) -> Button_Switch_Keyboard:SW_Cherry_MX_1.00u_Plate
- K_X1: renamed from K_X; footprint (none) -> Button_Switch_Keyboard:SW_Cherry_MX_1.00u_Plate
- K_Y1: renamed from K_Y; footprint (none) -> Button_Switch_Keyboard:SW_Cherry_MX_1.00u_Plate
- K_Z1: renamed from K_Z; footprint (none) -> Button_Switch_Keyboard:SW_Cherry_MX_1.00u_Plate
- K_[1: renamed from K_[; footprint (none) -> Button_Switch_Keyboard:SW_Cherry_MX_1.00u_Plate
- K_]1: renamed from K_]; footprint (none) -> Button_Switch_Keyboard:SW_Cherry_MX_1.00u_Plate
- gave numbers to parts that had none: 1

Commit message: Schematics Change
Wired all the microcontroller in schematics. Added Clock, Power Decoupler, ISP header, Reset switch, USB C connector
Parts:
- added C1, C2: 22p, Capacitor_SMD:C_0805_2012Metric, symbol Device:C_Small
- added C3: 1u, Capacitor_SMD:C_0805_2012Metric, symbol Device:C_Small
- added C4, C5, C6: 0.1u, Capacitor_SMD:C_0805_2012Metric, symbol Device:C_Small
- added C7: 10u, Capacitor_SMD:C_0805_2012Metric, symbol Device:C_Small
- added F1: 500m, Fuse:Fuse_1206_3216Metric_Pad1.42x1.75mm_HandSolder, symbol Device:Fuse_Small
- added J1: AVR-ISP-6, random-keyboard-parts:Reset_Pretty-Mask, symbol Connector:AVR-ISP-6
- added R1: 10k, Resistor_SMD:R_0805_2012Metric, symbol Device:R_Small
- added R2, R3: 5.1k, Resistor_SMD:R_0805_2012Metric, symbol Device:R_Small
- added R4: R, Resistor_SMD:R_0805_2012Metric, symbol Device:R
- added R6, R7: 22, Resistor_SMD:R_0805_2012Metric, symbol Device:R_Small
- added SW1: SW_PUSH, Button_Switch_SMD:SW_SPST_SKQG_WithStem, symbol keyboard_parts:SW_PUSH
- added U2: PRTR5V0U2X, random-keyboard-parts:SOT143B, symbol random-keyboard-parts:PRTR5V0U2X
- added USB1: HRO-TYPE-C-31-M-12, Type-C:HRO-TYPE-C-31-M-12-HandSoldering, symbol Type-C:HRO-TYPE-C-31-M-12
- added Y1: Crystal_GND24_Small, Crystal:Crystal_SMD_3225-4Pin_3.2x2.5mm, symbol Device:Crystal_GND24_Small
Connections:
- net Column 1: no longer D_#1.1 (K), D_'1.1 (K), D_,1.1 (K), D_-1.1 (K), D_.1.1 (K), D_/1.1 (K), D_0.1 (K), D_1.1 (K), D_2.1 (K), D_3.1 (K), D_4.1 (K), D_5.1 (K), D_6.1 (K), D_7.1 (K), D_8.1 (K), D_9.1 (K), D_;1.1 (K), D_=1.1 (K), D_A1.1 (K), D_ALT1.1 (K), D_ALT2.1 (K), D_B1.1 (K), D_BACK1.1 (K), D_C1.1 (K), D_CAPS1.1 (K), D_CTRL1.1 (K), D_D1.1 (K), D_DOWN1.1 (K), D_E1.1 (K), D_ENTER1.1 (K), D_ESC1.1 (K), D_F1.1 (K), D_FN1.1 (K), D_G1.1 (K), D_H1.1 (K), D_I1.1 (K), D_J1.1 (K), D_K1.1 (K), D_L1.1 (K), D_LEFT1.1 (K), D_M1.1 (K), D_MAC1.1 (K), D_MAC2.1 (K), D_MAC3.1 (K), D_MAC4.1 (K), D_MENU1.1 (K), D_N1.1 (K), D_O1.1 (K), D_P1.1 (K), D_Q1.1 (K), D_R1.1 (K), D_RIGHTY1.1 (K), D_S1.1 (K), D_SHIFT1.1 (K), D_SHIFT2.1 (K), D_SPACEBAR1.1 (K), D_T1.1 (K), D_TAB1.1 (K), D_U1.1 (K), D_UP1.1 (K), D_V1.1 (K), D_W1.1 (K), D_WINDOWS1.1 (K), D_X1.1 (K), D_Y1.1 (K), D_Z1.1 (K), D_[1.1 (K), D_]1.1 (K), K_#1.1, K_'1.1, K_,1.1, K_-1.1, K_.1.1, K_/1.1, K_0.1, K_1.1, K_2.1, K_3.1, K_4.1, K_5.1, K_6.1, K_7.1, K_8.1, K_9.1, K_;1.1, K_=1.1, K_A1.1, K_ALT1.1, K_ALT2.1, K_B1.1, K_BACK1.1, K_C1.1, K_CTRL2.1, K_D1.1, K_DOWN1.1, K_E1.1, K_ENTER1.1, K_F1.1, K_FN1.1, K_G1.1, K_H1.1, K_I1.1, K_J1.1, K_K1.1, K_L1.1, K_LEFT1.1, K_M1.1, K_MAC1.1, K_MAC2.1, K_MAC3.1, K_MAC4.1, K_N1.1, K_O1.1, K_P1.1, K_Q1.1, K_R1.1, K_RIGHT1.1, K_S1.1, K_SHIFT2.1, K_SPACEBARD1.1, K_T1.1, K_U1.1, K_UP1.1, K_V1.1, K_W1.1, K_WINDOWS1.1, K_X1.1, K_Y1.1, K_Z1.1, K_[1.1, K_]1.1, U1.25 (PD0), U1.26 (PD1), U1.32 (PD7), U1.33 (PE0), U1.34 (PE1), U1.35 (PC0), U1.36 (PC1), U1.37 (PC2), U1.38 (PC3), U1.39 (PC4), U1.40 (PC5), U1.41 (PC6), U1.42 (PC7), U1.43 (PE2/~{HWB}), U1.44 (PA7), U1.45 (PA6)
- net Column 2: now also K_1.1, K_A1.1, K_Q1.1, K_WINDOWS1.1, K_Z1.1
- net Row 3: now also D_'1.1 (K), D_;1.1 (K), D_A1.1 (K), D_CAPS1.1 (K), D_D1.1 (K), D_ENTER1.1 (K), D_F1.1 (K), D_G1.1 (K), D_H1.1 (K), D_J1.1 (K), D_K1.1 (K), D_L1.1 (K), D_S1.1 (K)
- net Row 4: now also D_,1.1 (K), D_.1.1 (K), D_/1.1 (K), D_B1.1 (K), D_C1.1 (K), D_M1.1 (K), D_N1.1 (K), D_SHIFT1.1 (K), D_SHIFT2.1 (K), D_UP1.1 (K), D_V1.1 (K), D_X1.1 (K), D_Z1.1 (K)
- net Row 5: now also D_ALT1.1 (K), D_ALT2.1 (K), D_CTRL1.1 (K), D_DOWN1.1 (K), D_FN1.1 (K), D_LEFT1.1 (K), D_MENU1.1 (K), D_RIGHTY1.1 (K), D_SPACEBAR1.1 (K), D_WINDOWS1.1 (K)
- net MISO: now reaches U1.10 (PB0)
- net MISO: now also J1.1 (MISO)
- net MOSI: now reaches U1.11 (PB1)
- net MOSI: now also J1.4 (MOSI)
- net SCK: now reaches U1.12 (PB2)
- net SCK: now also J1.3 (SCK)
- net RESET: now reaches U1.20 (~{RESET})
- net RESET: now also J1.5 (~{RST}), R4.2, SW1.2
- net +5V: now reaches U1.21 (VCC), U1.52 (VCC)
- net +5V: now also U1.22 (GND), U1.3 (UVCC), U1.53 (GND), U1.6 (UGND), U1.63 (GND), U1.64 (AVCC), U1.65 (GND), U1.8 (VBUS), C3.2, C4.1, C4.2, C5.1, C5.2, C6.1, C6.2, C7.1, C7.2, F1.2, J1.2 (VCC), J1.6 (GND), R1.2, R2.1, R3.1, R4.1, SW1.1, U2.1 (GND), USB1.1 (GND), USB1.12 (GND), USB1.13 (SHIELD), Y1.2, Y1.4
- net XTAL2: now reaches U1.23 (XTAL2)
- net XTAL2: now also C2.1, Y1.3
- net XTAL1: now reaches U1.24 (XTAL1)
- net XTAL1: now also C1.1, Y1.1
- net D-: now reaches U1.4 (D-)
- net D-: now also R6.2
- net Column 16: now reaches U1.46 (PA5)
- net Column 16: now also K_MAC2.1, K_MAC4.1, K_RIGHT1.1
- net D+: now reaches U1.5 (D+)
- net D+: now also R7.1
- net at U1.7 (UCAP): now also C3.1
- new net: R2.2, USB1.10 (CC2)
- new net: F1.1, USB1.11 (VBUS), USB1.2 (VBUS)
- new net: R3.2, USB1.4 (CC1)
- new net: R1.1, U1.43 (PE2/~{HWB})
- new net: C1.2, C2.2
- new net Column 10: K_.1.1, K_9.1, K_FN1.1, K_L1.1, K_O1.1, U1.39 (PC4)
- new net Column 11: K_/1.1, K_0.1, K_;1.1, K_CTRL2.1, K_P1.1, U1.40 (PC5)
- new net Column 12: K_'1.1, K_-1.1, K_LEFT1.1, K_SHIFT2.1, K_[1.1, U1.41 (PC6)
- new net Column 13: K_=1.1, K_ENTER1.1, K_]1.1, U1.42 (PC7)
- new net Column 14: K_#1.1, K_BACK1.1, U1.44 (PA7)
- new net Column 15: K_DOWN1.1, K_MAC1.1, K_MAC3.1, K_UP1.1, U1.45 (PA6)
- new net Column 3: K_2.1, K_ALT1.1, K_S1.1, K_W1.1, K_X1.1, U1.32 (PD7)
- new net Column 4: K_3.1, K_C1.1, K_D1.1, K_E1.1, U1.33 (PE0)
- new net Column 5: K_4.1, K_F1.1, K_R1.1, K_V1.1, U1.34 (PE1)
- new net Column 6: K_5.1, K_B1.1, K_G1.1, K_SPACEBARD1.1, K_T1.1, U1.35 (PC0)
- new net Column 7: K_6.1, K_H1.1, K_N1.1, K_Y1.1, U1.36 (PC1)
- new net Column 8: K_7.1, K_J1.1, K_M1.1, K_U1.1, U1.37 (PC2)
- new net Column 9: K_,1.1, K_8.1, K_ALT2.1, K_I1.1, K_K1.1, U1.38 (PC3)
- new net DN: R6.1, U2.3 (IO2), USB1.5 (DN2), USB1.7 (DN1)
- new net DP: R7.2, U2.2 (IO1), USB1.6 (DP1), USB1.8 (DP2)
- new net Row 1: D_-1.1 (K), D_0.1 (K), D_1.1 (K), D_2.1 (K), D_3.1 (K), D_4.1 (K), D_5.1 (K), D_6.1 (K), D_7.1 (K), D_8.1 (K), D_9.1 (K), D_=1.1 (K), D_BACK1.1 (K), D_ESC1.1 (K), D_MAC1.1 (K), D_MAC2.1 (K), U1.25 (PD0)
- new net Row 2: D_#1.1 (K), D_E1.1 (K), D_I1.1 (K), D_MAC3.1 (K), D_MAC4.1 (K), D_O1.1 (K), D_P1.1 (K), D_Q1.1 (K), D_R1.1 (K), D_T1.1 (K), D_TAB1.1 (K), D_U1.1 (K), D_W1.1 (K), D_Y1.1 (K), D_[1.1 (K), D_]1.1 (K), U1.26 (PD1)
- no-connect marks 0 -> 3
Other:
- moved on the sheet: U1
