File: Ki Cad PCB.kicad_pcb (KiCad board)
At the start: 2 copper layers, 337.6 x 98.6 mm, 138 parts, among them U1 AT90USB1286-M

Commit message: Updated pcb
Added all the traces for the pcb on while referring back to our switch matrix.
Parts:
- added C1: 22p, Capacitor_SMD:C_0805_2012Metric, F.Cu at (731.6, -147.1)
- added C2: 22p, Capacitor_SMD:C_0805_2012Metric, F.Cu at (736.0, -147.1)
- added C3: 1u, Capacitor_SMD:C_0805_2012Metric, F.Cu at (725.6, -140.8)
- added C4: 0.1u, Capacitor_SMD:C_0805_2012Metric, F.Cu at (723.5, -137.8)
- added C5: 0.1u, Capacitor_SMD:C_0805_2012Metric, F.Cu at (718.3, -132.0)
- added C6: 0.1u, Capacitor_SMD:C_0805_2012Metric, F.Cu at (725.6, -143.8)
- added C7: 10u, Capacitor_SMD:C_0805_2012Metric, F.Cu at (730.1, -143.8)
- added F1: 500m, Fuse:Fuse_1206_3216Metric_Pad1.42x1.75mm_HandSolder, F.Cu at (726.4, -146.9)
- added J1: AVR-ISP-6, random-keyboard-parts:Reset_Pretty-Mask, F.Cu at (720.3, -144.7)
- added R1: 10k, Resistor_SMD:R_0805_2012Metric, F.Cu at (722.7, -131.8)
- added R2: 5.1k, Resistor_SMD:R_0805_2012Metric, F.Cu at (728.0, -137.8)
- added R3: 5.1k, Resistor_SMD:R_0805_2012Metric, F.Cu at (730.1, -140.8)
- added R4: R, Resistor_SMD:R_0805_2012Metric, F.Cu at (728.0, -134.8)
- added R6: 22, Resistor_SMD:R_0805_2012Metric, F.Cu at (723.5, -134.8)
- added R7: 22, Resistor_SMD:R_0805_2012Metric, F.Cu at (734.5, -144.1)
- added SW1: SW_PUSH, Button_Switch_SMD:SW_SPST_SKQG_WithStem, F.Cu at (711.3, -134.5)
- added U2: PRTR5V0U2X, random-keyboard-parts:SOT143B, F.Cu at (734.3, -140.3)
- added USB1: HRO-TYPE-C-31-M-12, Type-C:HRO-TYPE-C-31-M-12-HandSoldering, F.Cu at (701.4, -139.9)
- added Y1: Crystal_GND24_Small, Crystal:Crystal_SMD_3225-4Pin_3.2x2.5mm, F.Cu at (718.7, -135.7)
- moved D_DOWN1 409.8 mm to (877.3, -1.28), turned to 180 degrees
- moved D_WINDOWS1 396.2 mm to (613.0, -0.88), turned to 180 degrees
- moved D_RIGHTY1 381.9 mm to (896.6, -1.18), turned to 180 degrees
- moved D_UP1 380.8 mm to (877.4, -19.9), turned to 180 degrees
- moved D_X1 368.9 mm to (648.9, -19.9), turned to 180 degrees
- moved D_CAPS1 366.5 mm to (594.1, -39.4), turned to 180 degrees
- moved U1 358.6 mm to (693.4, -100.3), turned to -90 degrees
- moved D_FN1 354.4 mm to (803.6, -1.28), turned to 180 degrees
- moved D_SPACEBAR1 349.8 mm to (707.8, -0.98), turned to 180 degrees
- moved D_ENTER1 349.5 mm to (841.9, -39.4), turned to 180 degrees
- moved D_,1 349.1 mm to (763.1, -20.2), turned to 180 degrees
- moved D_#1 348.6 mm to (848.7, -58.4), turned to 180 degrees
- moved D_SHIFT1 324.2 mm to (598.2, -20.3), turned to 180 degrees
- moved D_=1 318.2 mm to (815.2, -77.5), turned to 180 degrees
- moved D_ESC1 316.4 mm to (586.7, -77.5), turned to 180 degrees
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Connections:
- D_#1 pad 1: Column 1 -> Row 2
- D_'1 pad 1: Column 1 -> Row 3
- D_,1 pad 1: Column 1 -> Row 4
- D_-1 pad 1: Column 1 -> Row 1
- D_.1 pad 1: Column 1 -> Row 4
- D_/1 pad 1: Column 1 -> Row 4
- D_0 pad 1: Column 1 -> Row 1
- D_1 pad 1: Column 1 -> Row 1
- D_2 pad 1: Column 1 -> Row 1
- D_3 pad 1: Column 1 -> Row 1
- D_4 pad 1: Column 1 -> Row 1
- D_5 pad 1: Column 1 -> Row 1
- D_6 pad 1: Column 1 -> Row 1
- D_7 pad 1: Column 1 -> Row 1
- D_8 pad 1: Column 1 -> Row 1
- D_9 pad 1: Column 1 -> Row 1
- D_;1 pad 1: Column 1 -> Row 3
- D_=1 pad 1: Column 1 -> Row 1
- D_A1 pad 1: Column 1 -> Row 3
- D_ALT1 pad 1: Column 1 -> Row 5
- D_ALT2 pad 1: Column 1 -> Row 5
- D_B1 pad 1: Column 1 -> Row 4
- D_BACK1 pad 1: Column 1 -> Row 1
- D_C1 pad 1: Column 1 -> Row 4
- D_CAPS1 pad 1: Column 1 -> Row 3
- D_CTRL1 pad 1: Column 1 -> Row 5
- D_D1 pad 1: Column 1 -> Row 3
- D_DOWN1 pad 1: Column 1 -> Row 5
- D_E1 pad 1: Column 1 -> Row 2
- D_ENTER1 pad 1: Column 1 -> Row 3
- D_ESC1 pad 1: Column 1 -> Row 1
- D_F1 pad 1: Column 1 -> Row 3
- D_FN1 pad 1: Column 1 -> Row 5
- D_G1 pad 1: Column 1 -> Row 3
- D_H1 pad 1: Column 1 -> Row 3
- D_I1 pad 1: Column 1 -> Row 2
- D_J1 pad 1: Column 1 -> Row 3
- D_K1 pad 1: Column 1 -> Row 3
- D_L1 pad 1: Column 1 -> Row 3
- D_LEFT1 pad 1: Column 1 -> Row 5
- D_M1 pad 1: Column 1 -> Row 4
- D_MAC1 pad 1: Column 1 -> Row 1
- D_MAC2 pad 1: Column 1 -> Row 1
- D_MAC3 pad 1: Column 1 -> Row 2
- D_MAC4 pad 1: Column 1 -> Row 2
- D_MENU1 pad 1: Column 1 -> Row 5
- D_N1 pad 1: Column 1 -> Row 4
- D_O1 pad 1: Column 1 -> Row 2
- D_P1 pad 1: Column 1 -> Row 2
- D_Q1 pad 1: Column 1 -> Row 2
- D_R1 pad 1: Column 1 -> Row 2
- D_RIGHTY1 pad 1: Column 1 -> Row 5
- D_S1 pad 1: Column 1 -> Row 3
- D_SHIFT1 pad 1: Column 1 -> Row 4
- D_SHIFT2 pad 1: Column 1 -> Row 4
- D_SPACEBAR1 pad 1: Column 1 -> Row 5
- D_T1 pad 1: Column 1 -> Row 2
- D_TAB1 pad 1: Column 1 -> Row 2
- D_U1 pad 1: Column 1 -> Row 2
- D_UP1 pad 1: Column 1 -> Row 4
- D_V1 pad 1: Column 1 -> Row 4
- D_W1 pad 1: Column 1 -> Row 2
- D_WINDOWS1 pad 1: Column 1 -> Row 5
- D_X1 pad 1: Column 1 -> Row 4
- D_Y1 pad 1: Column 1 -> Row 2
- D_Z1 pad 1: Column 1 -> Row 4
- D_[1 pad 1: Column 1 -> Row 2
- D_]1 pad 1: Column 1 -> Row 2
- K_#1 pad 1: Column 1 -> Column 14
- K_'1 pad 1: Column 1 -> Column 12
- K_,1 pad 1: Column 1 -> Column 9
- K_-1 pad 1: Column 1 -> Column 12
- K_.1 pad 1: Column 1 -> Column 10
- K_/1 pad 1: Column 1 -> Column 11
- K_0 pad 1: Column 1 -> Column 11
- K_1 pad 1: Column 1 -> Column 2
- K_2 pad 1: Column 1 -> Column 3
- K_3 pad 1: Column 1 -> Column 4
- K_4 pad 1: Column 1 -> Column 5
- K_5 pad 1: Column 1 -> Column 6
- K_6 pad 1: Column 1 -> Column 7
- K_7 pad 1: Column 1 -> Column 8
- K_8 pad 1: Column 1 -> Column 9
- K_9 pad 1: Column 1 -> Column 10
- K_;1 pad 1: Column 1 -> Column 11
- K_=1 pad 1: Column 1 -> Column 13
- K_A1 pad 1: Column 1 -> Column 2
- K_ALT1 pad 1: Column 1 -> Column 3
- K_ALT2 pad 1: Column 1 -> Column 9
- K_B1 pad 1: Column 1 -> Column 6
- K_BACK1 pad 1: Column 1 -> Column 14
- K_C1 pad 1: Column 1 -> Column 4
- K_CTRL2 pad 1: Column 1 -> Column 11
- K_D1 pad 1: Column 1 -> Column 4
- K_DOWN1 pad 1: Column 1 -> Column 15
- K_E1 pad 1: Column 1 -> Column 4
- K_ENTER1 pad 1: Column 1 -> Column 13
- K_F1 pad 1: Column 1 -> Column 5
- K_FN1 pad 1: Column 1 -> Column 10
- K_G1 pad 1: Column 1 -> Column 6
- K_H1 pad 1: Column 1 -> Column 7
- K_I1 pad 1: Column 1 -> Column 9
- K_J1 pad 1: Column 1 -> Column 8
- K_K1 pad 1: Column 1 -> Column 9
- K_L1 pad 1: Column 1 -> Column 10
- K_LEFT1 pad 1: Column 1 -> Column 12
- K_M1 pad 1: Column 1 -> Column 8
- K_MAC1 pad 1: Column 1 -> Column 15
- K_MAC2 pad 1: Column 1 -> Column 16
- K_MAC3 pad 1: Column 1 -> Column 15
- K_MAC4 pad 1: Column 1 -> Column 16
- K_N1 pad 1: Column 1 -> Column 7
- K_O1 pad 1: Column 1 -> Column 10
- K_P1 pad 1: Column 1 -> Column 11
- K_Q1 pad 1: Column 1 -> Column 2
- K_R1 pad 1: Column 1 -> Column 5
- K_RIGHT1 pad 1: Column 1 -> Column 16
- K_S1 pad 1: Column 1 -> Column 3
- K_SHIFT2 pad 1: Column 1 -> Column 12
- K_SPACEBARD1 pad 1: Column 1 -> Column 6
- K_T1 pad 1: Column 1 -> Column 6
- K_U1 pad 1: Column 1 -> Column 8
- K_UP1 pad 1: Column 1 -> Column 15
- K_V1 pad 1: Column 1 -> Column 5
- K_W1 pad 1: Column 1 -> Column 3
- K_WINDOWS1 pad 1: Column 1 -> Column 2
- K_X1 pad 1: Column 1 -> Column 3
- K_Y1 pad 1: Column 1 -> Column 7
- K_Z1 pad 1: Column 1 -> Column 2
- K_[1 pad 1: Column 1 -> Column 12
- K_]1 pad 1: Column 1 -> Column 13
- U1 pad 10: unconnected-(U1-Pad10) -> MISO
- U1 pad 11: unconnected-(U1-Pad11) -> MOSI
- U1 pad 12: unconnected-(U1-Pad12) -> SCK
- U1 pad 20: unconnected-(U1-Pad20) -> RESET
- U1 pad 21: Net-(U1-Pad21) -> +5V
- U1 pad 22: Net-(U1-Pad22) -> +5V
- U1 pad 23: unconnected-(U1-Pad23) -> XTAL2
- U1 pad 24: unconnected-(U1-Pad24) -> XTAL1
- U1 pad 25: Column 1 -> Row 1
- U1 pad 26: Column 1 -> Row 2
- U1 pad 3: unconnected-(U1-Pad3) -> +5V
- U1 pad 32: Column 1 -> Column 3
- U1 pad 33: Column 1 -> Column 4
- U1 pad 34: Column 1 -> Column 5
- U1 pad 35: Column 1 -> Column 6
- U1 pad 36: Column 1 -> Column 7
- U1 pad 37: Column 1 -> Column 8
- U1 pad 38: Column 1 -> Column 9
- U1 pad 39: Column 1 -> Column 10
- U1 pad 4: unconnected-(U1-Pad4) -> D-
- U1 pad 40: Column 1 -> Column 11
- U1 pad 41: Column 1 -> Column 12
- U1 pad 42: Column 1 -> Column 13
- U1 pad 43: Column 1 -> Net-(R1-Pad1)
- U1 pad 44: Column 1 -> Column 14
- U1 pad 45: Column 1 -> Column 15
- U1 pad 46: unconnected-(U1-Pad46) -> Column 16
- U1 pad 5: unconnected-(U1-Pad5) -> D+
- U1 pad 52: Net-(U1-Pad21) -> +5V
- U1 pad 53: Net-(U1-Pad22) -> +5V
- U1 pad 6: unconnected-(U1-Pad6) -> +5V
- U1 pad 63: Net-(U1-Pad22) -> +5V
- U1 pad 64: unconnected-(U1-Pad64) -> +5V
- U1 pad 65: Net-(U1-Pad22) -> +5V
- U1 pad 7: unconnected-(U1-Pad7) -> Net-(C3-Pad1)
- U1 pad 8: unconnected-(U1-Pad8) -> +5V
Routing:
- net Row 5: track 0.00 -> 660.8 mm, vias 0 -> 1
- net Row 4: track 0.00 -> 647.1 mm, vias 0 -> 1
- net Row 2: track 0.00 -> 623.9 mm, vias 0 -> 2
- net Row 3: track 0.00 -> 596.9 mm, vias 0 -> 1
- net Row 1: track 0.00 -> 510.5 mm
- net Column 15: track 0.00 -> 345.2 mm
- net Column 16: track 0.00 -> 335.6 mm
- net Column 12: track 0.00 -> 302.3 mm
- net Column 1: track 0.00 -> 298.5 mm
- net Column 11: track 0.00 -> 293.5 mm
- net Column 2: track 0.00 -> 289.3 mm
- net Column 10: track 0.00 -> 271.8 mm
- net Column 3: track 0.00 -> 254.6 mm
- net Column 9: track 0.00 -> 248.1 mm
- net Column 13: track 0.00 -> 248.1 mm
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Other:
- board size 337.6 x 98.6 mm -> 327.6 x 120.6 mm
